Commit message: updated robot balance

File: Code/MuJoCo_SNS/robot_torso/ah001_manual_tree.urdf (robot description, URDF)
Before this commit: robot ah001_manual_tree, 15 links, 12 joints
Joints:
- added joint foot_l_passive_0: type fixed, parent shank_l, child foot_l, origin xyz=-0.12289387609137054 -0.29984794682384297 0.0075686485576649809 rpy=0 0 0, axis 0 0 0, limit effort=0 velocity=0
- added joint foot_r_passive_0: type fixed, parent shank_r, child foot_r, origin xyz=-0.08058292338752851 -0.31387591099248346 -0.013568653856787016 rpy=0 0 0, axis 0 0 0, limit effort=0 velocity=0
